Commit message: set imu rate param

File: xacro/realsense_d435i.xacro (robot description, xacro)
@@ -1,8 +1,6 @@
 <?xml version="1.0"?>
 <robot xmlns:xacro="http://www.ros.org/wiki/xacro">
-  <xacro:include filename="$(find realsense_ros_gazebo)/xacro/tracker.xacro"/>
-  <xacro:include filename="$(find realsense_ros_gazebo)/xacro/depthcam.xacro"/>
-  <xacro:macro name="realsense_d435i" params="sensor_name parent_link *origin rate">
-    <xacro:realsense_d435 sensor_name="${sensor_name}" parent_link="${parent_link}" rate="${rate}">
+  <xacro:macro name="realsense_d435i" params="sensor_name parent_link *origin image_rate imu_rate">
+    <xacro:realsense_d435 sensor_name="${sensor_name}" parent_link="${parent_link}" rate="${image_rate}">
       <xacro:insert_block name="origin" />
     </xacro:realsense_d435>
@@ -23,5 +21,5 @@
       <sensor name="imu_sensor" type="imu">
         <always_on>true</always_on>
-        <update_rate>400</update_rate>
+        <update_rate>${imu_rate}</update_rate>
         <visualize>true</visualize>
         <plugin name="imu_plugin" filename="libgazebo_ros_imu_sensor.so">
@@ -29,5 +27,5 @@
           <topicName>/${sensor_name}/imu</topicName>
           <bodyName>imu_link</bodyName>
-          <updateRateHZ>400.0</updateRateHZ>
+          <updateRateHZ>${imu_rate}</updateRateHZ>
           <gaussianNoise>0.0</gaussianNoise>
           <xyzOffset>0 0 0</xyzOffset>
