Commit message: change camera color

File: xacro/depthcam.xacro (robot description, xacro)
@@ -33,4 +33,7 @@
           <mesh filename="package://realsense_ros_gazebo/meshes/realsense_d435.stl" />
         </geometry>
+        <material name="white">
+            <color rgba="1.0 1.0 1.0 1.0" />
+        </material>
       </visual>
       <collision>
