Commit message: add realsense_d435i test

File: urdf/test.xacro (robot description, xacro)
@@ -3,4 +3,5 @@
   <xacro:include filename="$(find realsense_ros_gazebo)/xacro/tracker.xacro"/>
   <xacro:include filename="$(find realsense_ros_gazebo)/xacro/depthcam.xacro"/>
+  <xacro:include filename="$(find realsense_ros_gazebo)/xacro/realsense_d435i.xacro"/>
   <link name="base_footprint"/>
   <joint name="footprint_joint" type="fixed">
@@ -32,7 +33,10 @@
   </link>
   <!-- TEST -->
-  <xacro:realsense_d435 sensor_name="d435" parent_link="base_link" rate="10">
+  <xacro:realsense_d435i sensor_name="d435i" parent_link="base_link" image_rate="10" imu_rate="200">
     <origin rpy="0 0 0 " xyz="0 0 0.5"/>
-  </xacro:realsense_d435>
+  </xacro:realsense_d435i>
+  <!-- <xacro:realsense_d435 sensor_name="d435" parent_link="base_link" rate="10">
+    <origin rpy="0 0 0 " xyz="0 0 0.5"/>
+  </xacro:realsense_d435> -->
   <!-- <xacro:realsense_T265 sensor_name="camera" parent_link="base_link" rate="30.0">
     <origin rpy="0 0 0" xyz="0 0 0.5"/>
